Commit message: fix: change 23dof urdf & xml

File: humanoidverse/data/robots/x1/urdf/x1_23dof.urdf (robot description, URDF)
Before this commit: robot zhiyuan scene, 31 links, 30 joints
Joints:
- joint left_elbow_yaw_joint: type revolute -> fixed
- joint left_wrist_pitch_joint: type revolute -> fixed
- joint left_wrist_roll_joint: type revolute -> fixed
- joint right_elbow_yaw_joint: type revolute -> fixed
- joint right_wrist_pitch_joint: type revolute -> fixed
- joint right_wrist_roll_joint: type revolute -> fixed
