Commit message: fix: add para in asset & add new_urdf_rviz
humanoidverse/config/robot/x1/x1_29dof_leftleg.yaml

File: humanoidverse/data/robots/x1/urdf/x1.urdf (robot description, URDF)
Before this commit: robot zhiyuan scene, 31 links, 29 joints
Links:
- removed link link_left_knee_pitch
- added link link_lleft_knee_pitch, mass 1.68649; collision mesh filename=../meshes/left_knee_pitch.STL; visual mesh filename=../meshes/left_knee_pitch.STL
- link link_left_ankle_pitch: geometry collision mesh filename=../meshes/left_ankle_pitch.STL; visual mesh filename=../meshes/left_ankle_pitch.STL
- link link_left_ankle_roll: geometry collision mesh filename=../meshes/left_ankle_roll.STL; collision sphere radius=0.002
- link link_left_elbow_pitch: geometry collision mesh filename=../meshes/left_elbow_pitch.STL; visual mesh filename=../meshes/left_elbow_pitch.STL
- link link_left_elbow_yaw: geometry collision mesh filename=../meshes/left_elbow_yaw.STL; visual mesh filename=../meshes/left_elbow_yaw.STL
- link link_left_hip_pitch: geometry collision mesh filename=../meshes/left_hip_pitch.STL; visual mesh filename=../meshes/left_hip_pitch.STL
- link link_left_hip_roll: geometry collision mesh filename=../meshes/left_hip_roll.STL; visual mesh filename=../meshes/left_hip_roll.STL
- link link_left_hip_yaw: geometry collision mesh filename=../meshes/left_hip_yaw.STL; visual mesh filename=../meshes/left_hip_yaw.STL
- link link_left_shoulder_pitch: geometry collision mesh filename=../meshes/left_shoulder_pitch.STL; visual mesh filename=../meshes/left_shoulder_pitch.STL
- link link_left_shoulder_roll: geometry collision mesh filename=../meshes/left_shoulder_roll.STL; visual mesh filename=../meshes/left_shoulder_roll.STL
- link link_left_shoulder_yaw: geometry collision mesh filename=../meshes/left_shoulder_yaw.STL; visual mesh filename=../meshes/left_shoulder_yaw.STL
- link link_left_wrist_pitch: geometry collision mesh filename=../meshes/left_wrist_pitch.STL; visual mesh filename=../meshes/left_wrist_pitch.STL
- link link_left_wrist_roll: geometry collision mesh filename=../meshes/left_wrist_roll.STL; visual mesh filename=../meshes/left_wrist_roll.STL
- link link_lumbar_pitch: geometry collision mesh filename=../meshes/lumbar_pitch.STL; collision mesh filename=../meshes/lumbar_pitch.STL
- link link_lumbar_roll: geometry collision mesh filename=../meshes/lumbar_roll.STL; visual mesh filename=../meshes/lumbar_roll.STL
- link link_lumbar_yaw: geometry collision mesh filename=../meshes/lumbar_yaw.STL; visual mesh filename=../meshes/lumbar_yaw.STL
- link link_right_ankle_pitch: geometry collision mesh filename=../meshes/right_ankle_pitch.STL; visual mesh filename=../meshes/right_ankle_pitch.STL
- link link_right_ankle_roll: geometry collision mesh filename=../meshes/right_ankle_roll.STL; collision sphere radius=0.002
- link link_right_elbow_pitch: geometry collision mesh filename=../meshes/right_elbow_pitch.STL; visual mesh filename=../meshes/right_elbow_pitch.STL
- link link_right_elbow_yaw: geometry collision mesh filename=../meshes/right_elbow_yaw.STL; visual mesh filename=../meshes/right_elbow_yaw.STL
- link link_right_hip_pitch: geometry collision mesh filename=../meshes/right_hip_pitch.STL; visual mesh filename=../meshes/right_hip_pitch.STL
- link link_right_hip_roll: geometry collision mesh filename=../meshes/right_hip_roll.STL; visual mesh filename=../meshes/right_hip_roll.STL
- link link_right_hip_yaw: geometry collision mesh filename=../meshes/right_hip_yaw.STL; visual mesh filename=../meshes/right_hip_yaw.STL
- link link_right_knee_pitch: geometry collision mesh filename=../meshes/right_knee_pitch.STL; visual mesh filename=../meshes/right_knee_pitch.STL
- link link_right_shoulder_pitch: geometry collision mesh filename=../meshes/right_shoulder_pitch.STL; visual mesh filename=../meshes/right_shoulder_pitch.STL
- link link_right_shoulder_roll: geometry collision mesh filename=../meshes/right_shoulder_roll.STL; visual mesh filename=../meshes/right_shoulder_roll.STL
- link link_right_shoulder_yaw: geometry collision mesh filename=../meshes/right_shoulder_yaw.STL; visual mesh filename=../meshes/right_shoulder_yaw.STL
- link link_right_wrist_pitch: geometry collision mesh filename=../meshes/right_wrist_pitch.STL; visual mesh filename=../meshes/right_wrist_pitch.STL
- link link_right_wrist_roll: geometry collision mesh filename=../meshes/right_wrist_roll.STL; visual mesh filename=../meshes/right_wrist_roll.STL
- link x1-body: geometry collision mesh filename=../meshes/base_link_simple.STL; collision mesh filename=../meshes/base_link_simple.STL
Joints:
- added joint base_to_x1_body_joint: type fixed, parent base_link, child x1-body, origin xyz=0 0 0 rpy=0 0 0
- joint left_ankle_pitch_joint: parent link_left_knee_pitch -> link_lleft_knee_pitch
- joint left_knee_pitch_joint: child link_left_knee_pitch -> link_lleft_knee_pitch

Commit message: fix: fix lleft in urdf & xml
rm old version urdf

File: humanoidverse/data/robots/x1/urdf/x1.urdf (robot description, URDF)
Before this commit: robot zhiyuan scene, 31 links, 30 joints
Links:
- removed link link_lleft_knee_pitch
- added link link_left_knee_pitch, mass 1.68649; collision mesh filename=../meshes/left_knee_pitch.STL; visual mesh filename=../meshes/left_knee_pitch.STL
Joints:
- joint left_ankle_pitch_joint: parent link_lleft_knee_pitch -> link_left_knee_pitch
- joint left_knee_pitch_joint: child link_lleft_knee_pitch -> link_left_knee_pitch

Commit message: feat: change index order in urdf

File: humanoidverse/data/robots/x1/urdf/x1.urdf (robot description, URDF)
Before this commit: robot zhiyuan scene, 31 links, 30 joints
Joints:
- removed joint left_hip_pitch_joint
- added joint mleft_hip_pitch_joint: type revolute, parent x1-body, child link_left_hip_pitch, origin xyz=0.00245 0.092277 -0.012143 rpy=3.170218624440796e-07 -0.7853990876280905 1.570798162810677, axis 0 0 1, limit lower=-3.14 upper=6.28 effort=150.0 velocity=10

File: humanoidverse/data/robots/x1/urdf/x1_ros.urdf (robot description, URDF)
Before this commit: robot zhiyuan scene, 31 links, 30 joints
Joints:
- removed joint left_hip_pitch_joint
- added joint mleft_hip_pitch_joint: type revolute, parent x1-body, child link_left_hip_pitch, origin xyz=0.00245 0.092277 -0.012143 rpy=3.170218624440796e-07 -0.7853990876280905 1.570798162810677, axis 0 0 1, limit lower=-3.14 upper=6.28 effort=150.0 velocity=10

Commit message: feat: change urdf limit
version 2: lumbar, shoulder, hip, knee, ankle

File: humanoidverse/data/robots/x1/urdf/x1.urdf (robot description, URDF)
Before this commit: robot zhiyuan scene, 31 links, 30 joints
Joints:
- joint left_ankle_pitch_joint: limit lower=-1.0 upper=1.0 effort=18.0 velocity=10 -> lower=-0.87267 upper=0.5236 effort=18.0 velocity=10
- joint left_ankle_roll_joint: limit lower=-1.0 upper=1.0 effort=18.0 velocity=10 -> lower=-0.2618 upper=0.2618 effort=18.0 velocity=10
- joint left_hip_roll_joint: limit lower=-2.3 upper=0.8 effort=50.0 velocity=10 -> lower=-0.5236 upper=2.9671 effort=50.0 velocity=10
- joint left_hip_yaw_joint: limit lower=-3.14 upper=3.14 effort=50.0 velocity=10 -> lower=-2.7576 upper=2.7576 effort=50.0 velocity=10
- joint left_knee_pitch_joint: limit lower=0.0 upper=1.8 effort=150.0 velocity=10 -> lower=-0.087267 upper=2.8798 effort=150.0 velocity=10
- joint left_shoulder_pitch_joint: limit lower=-3.14 upper=3.14 effort=150.0 velocity=10 -> lower=-3.0892 upper=2.6704 effort=150.0 velocity=10
- joint left_shoulder_roll_joint: limit lower=-3.14 upper=0.0 effort=150.0 velocity=10 -> lower=-1.5882 upper=2.2515 effort=150.0 velocity=10
- joint left_shoulder_yaw_joint: limit lower=-3.14 upper=3.14 effort=150.0 velocity=10 -> lower=-2.618 upper=2.618 effort=150.0 velocity=10
- joint lumbar_yaw_joint: limit lower=-3.14 upper=3.14 effort=150.0 velocity=10 -> lower=-1 upper=1 effort=150.0 velocity=10
- joint mleft_hip_pitch_joint: limit lower=-3.14 upper=6.28 effort=150.0 velocity=10 -> lower=-2.5307 upper=2.8798 effort=150.0 velocity=10
- joint right_ankle_pitch_joint: limit lower=-1.0 upper=1.0 effort=18.0 velocity=10 -> lower=-0.87267 upper=0.5236 effort=18.0 velocity=10
- joint right_ankle_roll_joint: limit lower=-1.0 upper=1.0 effort=18.0 velocity=10 -> lower=-0.2618 upper=0.2618 effort=18.0 velocity=10
- joint right_hip_pitch_joint: limit lower=-6.28 upper=3.14 effort=150.0 velocity=10 -> lower=-2.5307 upper=2.8798 effort=150.0 velocity=10
- joint right_hip_roll_joint: limit lower=-0.8 upper=2.3 effort=50.0 velocity=10 -> lower=-2.9671 upper=0.5236 effort=50.0 velocity=10
- joint right_hip_yaw_joint: limit lower=-3.14 upper=3.14 effort=50.0 velocity=10 -> lower=-2.7576 upper=2.7576 effort=50.0 velocity=10
- joint right_knee_pitch_joint: limit lower=0.0 upper=1.8 effort=150.0 velocity=10 -> lower=-0.087267 upper=2.8798 effort=150.0 velocity=10
- joint right_shoulder_pitch_joint: limit lower=-3.14 upper=3.14 effort=150.0 velocity=10 -> lower=-3.0892 upper=2.6704 effort=150.0 velocity=10
- joint right_shoulder_roll_joint: limit lower=-3.14 upper=0.0 effort=150.0 velocity=10 -> lower=-2.2515 upper=1.5882 effort=150.0 velocity=10
- joint right_shoulder_yaw_joint: limit lower=-3.14 upper=3.14 effort=150.0 velocity=10 -> lower=-2.618 upper=2.618 effort=150.0 velocity=10

Commit message: feat: correct axis

File: humanoidverse/data/robots/x1/urdf/x1.urdf (robot description, URDF)
Before this commit: robot zhiyuan scene, 31 links, 30 joints
Joints:
- joint left_ankle_pitch_joint: limit lower=-0.87267 upper=0.5236 effort=18.0 velocity=10 -> lower=-0.1744 upper=0.1744 effort=18.0 velocity=10
- joint left_ankle_roll_joint: limit lower=-0.2618 upper=0.2618 effort=18.0 velocity=10 -> lower=-0.1744 upper=0.1744 effort=18.0 velocity=10
- joint left_hip_roll_joint: limit lower=-0.5236 upper=2.9671 effort=50.0 velocity=10 -> lower=-2.9671 upper=0.5236 effort=50.0 velocity=10
- joint left_shoulder_roll_joint: limit lower=-1.5882 upper=2.2515 effort=150.0 velocity=10 -> lower=-2.2515 upper=0 effort=150.0 velocity=10
- joint mleft_hip_pitch_joint: limit lower=-2.5307 upper=2.8798 effort=150.0 velocity=10 -> lower=-2.8798 upper=2.5307 effort=150.0 velocity=10
- joint right_ankle_pitch_joint: limit lower=-0.87267 upper=0.5236 effort=18.0 velocity=10 -> lower=-0.1744 upper=0.1744 effort=18.0 velocity=10
- joint right_ankle_roll_joint: limit lower=-0.2618 upper=0.2618 effort=18.0 velocity=10 -> lower=-0.1744 upper=0.1744 effort=18.0 velocity=10
- joint right_hip_roll_joint: limit lower=-2.9671 upper=0.5236 effort=50.0 velocity=10 -> lower=-0.5236 upper=2.9671 effort=50.0 velocity=10
- joint right_shoulder_roll_joint: limit lower=-2.2515 upper=1.5882 effort=150.0 velocity=10 -> lower=-2.2515 upper=0.0 effort=150.0 velocity=10

Commit message: dev: sync shoulder_pitch_joint limit ref to real
- humanoidverse\config\robot\x1\x1_29dof.yaml
- humanoidverse\data\robots\x1\urdf\x1.urdf

File: humanoidverse/data/robots/x1/urdf/x1.urdf (robot description, URDF)
Before this commit: robot zhiyuan scene, 31 links, 30 joints
Joints:
- joint left_shoulder_pitch_joint: limit lower=-3.0892 upper=2.6704 effort=150.0 velocity=10 -> lower=-3.0892 upper=1.0467 effort=150.0 velocity=10
- joint right_shoulder_pitch_joint: limit lower=-3.0892 upper=2.6704 effort=150.0 velocity=10 -> lower=-3.0892 upper=1.0467 effort=150.0 velocity=10
